Commit message: gazebo plugin

File: description/rosbot.urdf.xacro (robot description, xacro)
@@ -2,3 +2,4 @@
 <robot xmlns:xacro="http://www.ros.org/wiki/xacro"  name="robot">
     <xacro:include filename="rosbot_core.xacro" />
+    <xacro:include filename="rosbot_control.xacro" />
 </robot>

File: description/rosbot_core.xacro (robot description, xacro)
@@ -1,4 +1,6 @@
 <?xml version="1.0"?>
 <robot xmlns:xacro="http://www.ros.org/wiki/xacro">
+    <xacro:arg name="mesh_path" default="${mesh_path}" />
+    <xacro:property name="mesh_path" value="$(arg mesh_path)" />
     <material name="white">
         <color rgba="1 1 1 1" />
@@ -14,5 +16,5 @@
     </material>
     <link
-    name="base_link">
+        name="base_link">
         <inertial>
             <origin
@@ -35,19 +37,17 @@
             <geometry>
                 <mesh
-                    filename="package://rosbot/description/meshes/base_link.STL" />
-            </geometry>
-            <material
-                name="">
-                <color
-                    rgba="0.79216 0.81961 0.93333 1" />
-            </material>
-        </visual>
-        <collision>
-            <origin
-                xyz="0 0 0"
-                rpy="0 0 0" />
-            <geometry>
-                <mesh
-                    filename="package://rosbot/description/meshes/base_link.STL" />
+                    filename="${mesh_path}base_link.STL" />
+            </geometry>
+            <material name="white">
+                <color rgba="1 1 1 1" />
+            </material>
+        </visual>
+        <collision>
+            <origin
+                xyz="0 0 0"
+                rpy="0 0 0" />
+            <geometry>
+                <mesh
+                    filename="${mesh_path}base_link.STL" />
             </geometry>
         </collision>
@@ -75,19 +75,17 @@
             <geometry>
                 <mesh
-                    filename="package://rosbot/description/meshes/fl_wheel_Link.STL" />
-            </geometry>
-            <material
-                name="">
-                <color
-                    rgba="0.792156862745098 0.819607843137255 0.933333333333333 1" />
-            </material>
-        </visual>
-        <collision>
-            <origin
-                xyz="0 0 0"
-                rpy="0 0 0" />
-            <geometry>
-                <mesh
-                    filename="package://rosbot/description/meshes/fl_wheel_Link.STL" />
+                    filename="${mesh_path}fl_wheel_Link.STL" />
+            </geometry>
+            <material name="black">
+                <color rgba="0 0 0 1" />
+            </material>
+        </visual>
+        <collision>
+            <origin
+                xyz="0 0 0"
+                rpy="0 0 0" />
+            <geometry>
+                <mesh
+                    filename="${mesh_path}fl_wheel_Link.STL" />
             </geometry>
         </collision>
@@ -128,19 +126,17 @@
             <geometry>
                 <mesh
-                    filename="package://rosbot/description/meshes/bl_wheel_Link.STL" />
-            </geometry>
-            <material
-                name="">
-                <color
-                    rgba="0.792156862745098 0.819607843137255 0.933333333333333 1" />
-            </material>
-        </visual>
-        <collision>
-            <origin
-                xyz="0 0 0"
-                rpy="0 0 0" />
-            <geometry>
-                <mesh
-                    filename="package://rosbot/description/meshes/bl_wheel_Link.STL" />
+                    filename="${mesh_path}bl_wheel_Link.STL" />
+            </geometry>
+            <material name="black">
+                <color rgba="0 0 0 1" />
+            </material>
+        </visual>
+        <collision>
+            <origin
+                xyz="0 0 0"
+                rpy="0 0 0" />
+            <geometry>
+                <mesh
+                    filename="${mesh_path}bl_wheel_Link.STL" />
             </geometry>
         </collision>
@@ -181,19 +177,17 @@
             <geometry>
                 <mesh
-                    filename="package://rosbot/description/meshes/fr_wheel_Link.STL" />
-            </geometry>
-            <material
-                name="">
-                <color
-                    rgba="0.792156862745098 0.819607843137255 0.933333333333333 1" />
-            </material>
-        </visual>
-        <collision>
-            <origin
-                xyz="0 0 0"
-                rpy="0 0 0" />
-            <geometry>
-                <mesh
-                    filename="package://rosbot/description/meshes/fr_wheel_Link.STL" />
+                    filename="${mesh_path}fr_wheel_Link.STL" />
+            </geometry>
+            <material name="black">
+                <color rgba="0 0 0 1" />
+            </material>
+        </visual>
+        <collision>
+            <origin
+                xyz="0 0 0"
+                rpy="0 0 0" />
+            <geometry>
+                <mesh
+                    filename="${mesh_path}fr_wheel_Link.STL" />
             </geometry>
         </collision>
@@ -234,19 +228,17 @@
             <geometry>
                 <mesh
-                    filename="package://rosbot/description/meshes/br_wheel_Link.STL" />
-            </geometry>
-            <material
-                name="">
-                <color
-                    rgba="0.792156862745098 0.819607843137255 0.933333333333333 1" />
-            </material>
-        </visual>
-        <collision>
-            <origin
-                xyz="0 0 0"
-                rpy="0 0 0" />
-            <geometry>
-                <mesh
-                    filename="package://rosbot/description/meshes/br_wheel_Link.STL" />
+                    filename="${mesh_path}br_wheel_Link.STL" />
+            </geometry>
+            <material name="black">
+                <color rgba="0 0 0 1" />
+            </material>
+        </visual>
+        <collision>
+            <origin
+                xyz="0 0 0"
+                rpy="0 0 0" />
+            <geometry>
+                <mesh
+                    filename="${mesh_path}br_wheel_Link.STL" />
             </geometry>
         </collision>
@@ -287,19 +279,17 @@
             <geometry>
                 <mesh
-                    filename="package://rosbot/description/meshes/lidar_Link.STL" />
-            </geometry>
-            <material
-                name="">
-                <color
-                    rgba="0.752941176470588 0.752941176470588 0.752941176470588 0.4" />
-            </material>
-        </visual>
-        <collision>
-            <origin
-                xyz="0 0 0"
-                rpy="0 0 0" />
-            <geometry>
-                <mesh
-                    filename="package://rosbot/description/meshes/lidar_Link.STL" />
+                    filename="${mesh_path}lidar_Link.STL" />
+            </geometry>
+            <material name="light_purple">
+                <color rgba="0.8 0.6 1.0 1" />
+            </material>
+        </visual>
+        <collision>
+            <origin
+                xyz="0 0 0"
+                rpy="0 0 0" />
+            <geometry>
+                <mesh
+                    filename="${mesh_path}lidar_Link.STL" />
             </geometry>
         </collision>
@@ -340,19 +330,17 @@
             <geometry>
                 <mesh
-                    filename="package://rosbot/description/meshes/camera_Link.STL" />
-            </geometry>
-            <material
-                name="">
-                <color
-                    rgba="1 1 1 1" />
-            </material>
-        </visual>
-        <collision>
-            <origin
-                xyz="0 0 0"
-                rpy="0 0 0" />
-            <geometry>
-                <mesh
-                    filename="package://rosbot/description/meshes/camera_Link.STL" />
+                    filename="${mesh_path}camera_Link.STL" />
+            </geometry>
+            <material name="light_green">
+                <color rgba="0.6 1.0 0.6 1" />
+            </material>
+        </visual>
+        <collision>
+            <origin
+                xyz="0 0 0"
+                rpy="0 0 0" />
+            <geometry>
+                <mesh
+                    filename="${mesh_path}camera_Link.STL" />
             </geometry>
         </collision>

Commit message: base and wheels

File: description/rosbot.urdf.xacro (robot description, xacro)
@@ -2,4 +2,4 @@
 <robot xmlns:xacro="http://www.ros.org/wiki/xacro"  name="robot">
     <xacro:include filename="rosbot_core.xacro" />
-    <xacro:include filename="rosbot_control.xacro" />
+    <!-- <xacro:include filename="rosbot_control.xacro" /> -->
 </robot>

File: description/rosbot_control.xacro (robot description, xacro)
@@ -1,3 +1,3 @@
-<?xml version="1.0"?>
+<!-- <?xml version="1.0"?>
 <robot xmlns:xacro="http://www.ros.org/wiki/xacro">
     <gazebo>
@@ -15,3 +15,3 @@
         </plugin>
     </gazebo>
-</robot>
+</robot> -->

File: description/rosbot_core.xacro (robot description, xacro)
@@ -15,4 +15,14 @@
         <color rgba="0 0 0 1" />
     </material>
+    <!-- Base footprint - virtual link on the ground plane -->
+    <link name="base_footprint">
+        <!-- No inertial, visual, or collision properties needed -->
+    </link>
+    <!-- Joint connecting base_footprint to base_link -->
+    <joint name="base_footprint_joint" type="fixed">
+        <origin xyz="0 0 0.015" rpy="0 0 0" />  <!-- Adjust Z based on your wheel radius -->
+        <parent link="base_footprint" />
+        <child link="base_link" />
+    </joint>
     <link
         name="base_link">
@@ -105,4 +115,55 @@
     </joint>
     <link
+        name="fr_wheel_Link">
+        <inertial>
+            <origin
+                xyz="-2.21104246023174E-10 -7.2173080359339E-10 0.00153990830645513"
+                rpy="0 0 0" />
+            <mass
+                value="0.0351743525851942" />
+            <inertia
+                ixx="1.52368217807294E-05"
+                ixy="-4.78967548245282E-10"
+                ixz="1.3714121636048E-13"
+                iyy="1.52370860963441E-05"
+                iyz="-2.12345782810308E-14"
+                izz="2.57855729883382E-05" />
+        </inertial>
+        <visual>
+            <origin
+                xyz="0 0 0"
+                rpy="0 0 0" />
+            <geometry>
+                <mesh
+                    filename="${mesh_path}fr_wheel_Link.STL" />
+            </geometry>
+            <material name="black">
+                <color rgba="0 0 0 1" />
+            </material>
+        </visual>
+        <collision>
+            <origin
+                xyz="0 0 0"
+                rpy="0 0 0" />
+            <geometry>
+                <mesh
+                    filename="${mesh_path}fr_wheel_Link.STL" />
+            </geometry>
+        </collision>
+    </link>
+    <joint
+        name="fr_wheel_joint"
+        type="continuous">
+        <origin
+            xyz="0.054819 -0.11375 0.0125"
+            rpy="-1.5708 0 0" />
+        <parent
+            link="base_link" />
+        <child
+            link="fr_wheel_Link" />
+        <axis
+            xyz="0 0 -1" />
+    </joint>
+    <link
         name="bl_wheel_Link">
         <inertial>
@@ -156,55 +217,4 @@
     </joint>
     <link
-        name="fr_wheel_Link">
-        <inertial>
-            <origin
-                xyz="-2.21104246023174E-10 -7.2173080359339E-10 0.00153990830645513"
-                rpy="0 0 0" />
-            <mass
-                value="0.0351743525851942" />
-            <inertia
-                ixx="1.52368217807294E-05"
-                ixy="-4.78967548245282E-10"
-                ixz="1.3714121636048E-13"
-                iyy="1.52370860963441E-05"
-                iyz="-2.12345782810308E-14"
-                izz="2.57855729883382E-05" />
-        </inertial>
-        <visual>
-            <origin
-                xyz="0 0 0"
-                rpy="0 0 0" />
-            <geometry>
-                <mesh
-                    filename="${mesh_path}fr_wheel_Link.STL" />
-            </geometry>
-            <material name="black">
-                <color rgba="0 0 0 1" />
-            </material>
-        </visual>
-        <collision>
-            <origin
-                xyz="0 0 0"
-                rpy="0 0 0" />
-            <geometry>
-                <mesh
-                    filename="${mesh_path}fr_wheel_Link.STL" />
-            </geometry>
-        </collision>
-    </link>
-    <joint
-        name="fr_wheel_joint"
-        type="continuous">
-        <origin
-            xyz="0.054819 -0.11375 0.0125"
-            rpy="-1.5708 0 0" />
-        <parent
-            link="base_link" />
-        <child
-            link="fr_wheel_Link" />
-        <axis
-            xyz="0 0 -1" />
-    </joint>
-    <link
         name="br_wheel_Link">
         <inertial>
@@ -257,5 +267,5 @@
             xyz="0 0 -1" />
     </joint>
-    <link
+    <!-- <link
         name="lidar_Link">
         <inertial>
@@ -307,6 +317,6 @@
         <axis
             xyz="0 0 1" />
-    </joint>
-    <link
+    </joint> -->
+    <!-- <link
         name="camera_Link">
         <inertial>
@@ -358,4 +368,4 @@
         <axis
             xyz="0 0 0" />
-    </joint>
+    </joint> -->
 </robot>

Commit message: movement done

File: description/rosbot.urdf.xacro (robot description, xacro)
@@ -1,5 +1,9 @@
-<?xml version="1.0"?>
-<robot xmlns:xacro="http://www.ros.org/wiki/xacro"  name="robot">
-    <xacro:include filename="rosbot_core.xacro" />
-    <!-- <xacro:include filename="rosbot_control.xacro" /> -->
+<robot xmlns:xacro="http://www.ros.org/wiki/xacro" name="rosbot">
+  <xacro:arg name="sim_mode" default="true" />
+  <xacro:arg name="mesh_path" default="$(find rosbot)/description/meshes" />
+  <!-- ✅ Just include raw XML -->
+  <xacro:include filename="$(find rosbot)/description/rosbot_core.xacro" />
+  <xacro:include filename="$(find rosbot)/description/rosbot_control.xacro" />
+  <xacro:include filename="$(find rosbot)/description/lidar.xacro" />
+  <xacro:include filename="$(find rosbot)/description/camera.xacro" />
 </robot>

File: description/rosbot_control.xacro (robot description, xacro)
@@ -1,17 +1,42 @@
-<!-- <?xml version="1.0"?>
+<?xml version="1.0"?>
 <robot xmlns:xacro="http://www.ros.org/wiki/xacro">
     <gazebo>
-        <plugin name="ros2_diff_drive" filename="libros_gz_diff_drive_system.so">
-            <left_joint>fl_wheel_joint</left_joint>
-            <right_joint>fr_wheel_joint</right_joint>
-            <wheel_separation>0.2275</wheel_separation>
-            <wheel_radius>0.0125</wheel_radius>
-            <odometry_frame>odom</odometry_frame>
-            <robot_base_frame>base_link</robot_base_frame>
-            <topic>cmd_vel</topic>
-            <odometry_topic>odom</odometry_topic>
-            <publish_odom>true</publish_odom>
-            <publish_tf>true</publish_tf>
+        <plugin name="ros2_control" filename="libgz_ros2_control-system.so">
+            <robot_param>robot_description</robot_param>
         </plugin>
     </gazebo>
-</robot> -->
+    <ros2_control name="GazeboSystem" type="system">
+        <hardware>
+            <plugin>gazebo_ros2_control/GazeboSystem</plugin>
+        </hardware>
+        <joint name="fl_wheel_joint">
+            <command_interface name="velocity" />
+            <state_interface name="velocity" />
+            <state_interface name="position" />
+        </joint>
+        <joint name="fr_wheel_joint">
+            <command_interface name="velocity" />
+            <state_interface name="velocity" />
+            <state_interface name="position" />
+        </joint>
+        <joint name="bl_wheel_joint">
+            <command_interface name="velocity" />
+            <state_interface name="velocity" />
+            <state_interface name="position" />
+        </joint>
+        <joint name="br_wheel_joint">
+            <command_interface name="velocity" />
+            <state_interface name="velocity" />
+            <state_interface name="position" />
+        </joint>
+    </ros2_control>
+    <transmission name="fl_wheel_trans">
+        <type>transmission_interface/SimpleTransmission</type>
+        <joint name="fl_wheel_joint">
+            <hardwareInterface>hardware_interface/VelocityJointInterface</hardwareInterface>
+        </joint>
+        <actuator name="fl_wheel_motor">
+            <hardwareInterface>hardware_interface/VelocityJointInterface</hardwareInterface>
+        </actuator>
+    </transmission>
+</robot>

File: description/rosbot_core.xacro (robot description, xacro)
@@ -1,6 +1,6 @@
 <?xml version="1.0"?>
 <robot xmlns:xacro="http://www.ros.org/wiki/xacro">
-    <xacro:arg name="mesh_path" default="${mesh_path}" />
-    <xacro:property name="mesh_path" value="$(arg mesh_path)" />
+    <xacro:property name="mesh_path" value="$(find rosbot)/description/meshes" />
+    <xacro:arg name="sim_mode" default="true" />
     <material name="white">
         <color rgba="1 1 1 1" />
@@ -21,5 +21,5 @@
     <!-- Joint connecting base_footprint to base_link -->
     <joint name="base_footprint_joint" type="fixed">
-        <origin xyz="0 0 0.015" rpy="0 0 0" />  <!-- Adjust Z based on your wheel radius -->
+        <origin xyz="0 0 0.0325" rpy="0 0 0" />  <!-- Adjust Z based on your wheel radius -->
         <parent link="base_footprint" />
         <child link="base_link" />
@@ -47,5 +47,5 @@
             <geometry>
                 <mesh
-                    filename="${mesh_path}base_link.STL" />
+                    filename="${mesh_path}/base_link.STL" />
             </geometry>
             <material name="white">
@@ -59,5 +59,5 @@
             <geometry>
                 <mesh
-                    filename="${mesh_path}base_link.STL" />
+                    filename="${mesh_path}/base_link.STL" />
             </geometry>
         </collision>
@@ -85,5 +85,5 @@
             <geometry>
                 <mesh
-                    filename="${mesh_path}fl_wheel_Link.STL" />
+                    filename="${mesh_path}/fl_wheel_Link.STL" />
             </geometry>
             <material name="black">
@@ -97,5 +97,5 @@
             <geometry>
                 <mesh
-                    filename="${mesh_path}fl_wheel_Link.STL" />
+                    filename="${mesh_path}/fl_wheel_Link.STL" />
             </geometry>
         </collision>
@@ -105,5 +105,5 @@
         type="continuous">
         <origin
-            xyz="0.054819 0.11375 0.0125"
+            xyz="0.054819 0.11375 0.0325"
             rpy="1.5708 0 0" />
         <parent
@@ -136,5 +136,5 @@
             <geometry>
                 <mesh
-                    filename="${mesh_path}fr_wheel_Link.STL" />
+                    filename="${mesh_path}/fr_wheel_Link.STL" />
             </geometry>
             <material name="black">
@@ -148,5 +148,5 @@
             <geometry>
                 <mesh
-                    filename="${mesh_path}fr_wheel_Link.STL" />
+                    filename="${mesh_path}/fr_wheel_Link.STL" />
             </geometry>
         </collision>
@@ -156,5 +156,5 @@
         type="continuous">
         <origin
-            xyz="0.054819 -0.11375 0.0125"
+            xyz="0.054819 -0.11375 0.0325"
             rpy="-1.5708 0 0" />
         <parent
@@ -187,5 +187,5 @@
             <geometry>
                 <mesh
-                    filename="${mesh_path}bl_wheel_Link.STL" />
+                    filename="${mesh_path}/bl_wheel_Link.STL" />
             </geometry>
             <material name="black">
@@ -199,5 +199,5 @@
             <geometry>
                 <mesh
-                    filename="${mesh_path}bl_wheel_Link.STL" />
+                    filename="${mesh_path}/bl_wheel_Link.STL" />
             </geometry>
         </collision>
@@ -207,5 +207,5 @@
         type="continuous">
         <origin
-            xyz="-0.064819 0.11375 0.0125"
+            xyz="-0.064819 0.11375 0.0325"
             rpy="1.5708 0 0" />
         <parent
@@ -238,5 +238,5 @@
             <geometry>
                 <mesh
-                    filename="${mesh_path}br_wheel_Link.STL" />
+                    filename="${mesh_path}/br_wheel_Link.STL" />
             </geometry>
             <material name="black">
@@ -250,5 +250,5 @@
             <geometry>
                 <mesh
-                    filename="${mesh_path}br_wheel_Link.STL" />
+                    filename="${mesh_path}/br_wheel_Link.STL" />
             </geometry>
         </collision>
@@ -258,5 +258,5 @@
         type="continuous">
         <origin
-            xyz="-0.064819 -0.11375 0.0125"
+            xyz="-0.064819 -0.11375 0.0325"
             rpy="-1.5708 0 0" />
         <parent
@@ -289,5 +289,5 @@
             <geometry>
                 <mesh
-                    filename="${mesh_path}lidar_Link.STL" />
+                    filename="${mesh_path}/lidar_Link.STL" />
             </geometry>
             <material name="light_purple">
@@ -301,5 +301,5 @@
             <geometry>
                 <mesh
-                    filename="${mesh_path}lidar_Link.STL" />
+                    filename="${mesh_path}/lidar_Link.STL" />
             </geometry>
         </collision>
@@ -340,5 +340,5 @@
             <geometry>
                 <mesh
-                    filename="${mesh_path}camera_Link.STL" />
+                    filename="${mesh_path}/camera_Link.STL" />
             </geometry>
             <material name="light_green">
@@ -352,5 +352,5 @@
             <geometry>
                 <mesh
-                    filename="${mesh_path}camera_Link.STL" />
+                    filename="${mesh_path}/camera_Link.STL" />
             </geometry>
         </collision>
